File: diplom.sch (KiCad schematic (older format))
At the start: 124 parts, among them J1 USB_B, J2 Barrel_Jack, J3 USB_B, J4 Screw_Terminal_01x03, J5 Screw_Terminal_01x04, J6 Screw_Terminal_01x04, J7 Screw_Terminal_01x04, J8 Screw_Terminal_01x02, Q1 S8050, SW1 SW_Push, SW2 SW_SPST, SW3 SW_SPDT, SW4 SW_SPDT, SW5 SW_Push, SW6 SW_Push, SW7 SW_Push, SW8 SW_Push, U1 LD3985M33R, U10 L298, U11 LS7366R, U12 LS7366R, U2 TPS54620, U3 STM32F103_STLINK, U4 CP2102, U5 TPS76833, U6 STM32F446, U7 STM32F103_DC, U8 TCA9517, U9 PCF8574, Y1 8MHz, Y2 8MHz, Y3 20MHz, Y4 20MHz

Commit message: Schematic redraw. Wire redrawing for correctness
Parts:
- removed C16, C17, C18, C35, C8: 100n, Capacitors_SMD:C_0603_HandSoldering, symbol C
- removed C19: 0.1u, Capacitors_SMD:C_0603_HandSoldering, symbol C
- removed C34: 1u, Capacitors_SMD:C_1210_HandSoldering, symbol CP
- removed C40, C5, C6: 20p, Capacitors_SMD:C_0603_HandSoldering, symbol C
- removed D2: LED, Diodes_SMD:D_0805, symbol LED
- removed J1, J3: USB_B, Connectors_USB:USB_Micro-B_Molex_47346-0001, symbol USB_B-RESCUE-diplom
- removed J4: Screw_Terminal_01x03, Pin_Headers:Pin_Header_Straight_1x03_Pitch2.54mm, symbol Screw_Terminal_01x03
- removed R1: 1K5, Resistors_SMD:R_0603_HandSoldering, symbol R
- removed R2, R4: 100K, Resistors_SMD:R_0603_HandSoldering, symbol R
- removed R6: 2K2, Resistors_SMD:R_0603_HandSoldering, symbol R
- removed R8: 10K, Resistors_SMD:R_0603_HandSoldering, symbol R
- removed R9: 4K7, Resistors_SMD:R_0603_HandSoldering, symbol R
- removed SW2: SW_SPST, Pin_Headers:Pin_Header_Straight_1x03_Pitch2.54mm, symbol SW_SPST-RESCUE-diplom
- removed SW3, SW4: SW_SPDT, Pin_Headers:Pin_Header_Straight_1x03_Pitch2.54mm, symbol SW_SPDT
- removed U3: STM32F103_STLINK, Housings_QFP:LQFP-48_7x7mm_Pitch0.5mm, symbol STM32F103_STLINK
- removed Y1: 8MHz, Crystals:Crystal_SMD_EuroQuartz_MQ2-2pin_7.0x5.0mm_HandSoldering, symbol Crystal
- added C34, C? (x5): 100n, Capacitors_SMD:C_0603_HandSoldering, symbol C
- added C35: 1u, Capacitors_SMD:C_1210_HandSoldering, symbol CP
- added C42, C? (x2): 20p, Capacitors_SMD:C_0603_HandSoldering, symbol C
- added D?: LED, Diodes_SMD:D_0805, symbol LED
- added J3, J?: USB_B, symbol USB_B
- added J?: Screw_Terminal_01x03, Pin_Headers:Pin_Header_Straight_1x03_Pitch2.54mm, symbol Screw_Terminal_01x03
- added R?: 2K2, Resistors_SMD:R_0603_HandSoldering, symbol R
- added R? (x2): 4K7, Resistors_SMD:R_0603_HandSoldering, symbol R
- added R? (x2): 100K, Resistors_SMD:R_0603_HandSoldering, symbol R
- added R?: 1K5, Resistors_SMD:R_0603_HandSoldering, symbol R
- added SW2: SW_SPST, Pin_Headers:Pin_Header_Straight_1x03_Pitch2.54mm, symbol SW_SPST
- added SW? (x2): SW_SPDT, Pin_Headers:Pin_Header_Straight_1x03_Pitch2.54mm, symbol SW_SPDT
- added U?: STM32F103_STLINK, Housings_QFP:LQFP-48_7x7mm_Pitch0.5mm, symbol STM32F103_STLINK
- added Y?: 8MHz, Crystals:Crystal_SMD_EuroQuartz_MQ2-2pin_7.0x5.0mm_HandSoldering, symbol Crystal
- C20: value 100n -> 0.1u
- C31: value 100n -> 10u; footprint Capacitors_SMD:C_0603_HandSoldering -> Capacitors_SMD:C_1206_HandSoldering
- C32: value 10u -> 100n; footprint Capacitors_SMD:C_1206_HandSoldering -> Capacitors_SMD:C_0603_HandSoldering
- C36: value 4.7u -> 100n; footprint Capacitors_SMD:C_0805_HandSoldering -> Capacitors_SMD:C_0603_HandSoldering
- C37: value 100n -> 4.7u; footprint Capacitors_SMD:C_0603_HandSoldering -> Capacitors_SMD:C_0805_HandSoldering
- R10: value 4K7 -> 52K5
- R11, R20: value 2K2 -> 10K
- R18: value 10K -> 100K
- R19: value 100K -> 2K2
- R7: value 52K5 -> 2K2
- renumbered C42 to C40
Connections:
- net +12V: now also C13.1, D1.1 (K)
- net +3.3VA: now also C?.1, C?.1, C?.1, C?.1, D?.2 (A), R?.1, R?.2, R?.2, U?.1 (BAT), U?.24 (VDD), U?.36 (VDD), U?.48 (VDD), U?.9 (VDDA); no longer C20.1
- net +3V3: now also C33.1, C36.1, R19.2, R20.2, R21.2, C34.1; no longer C30.1, C37.1, R18.2, R21.1, R22.1
- net +5V: now also R10.2; no longer R7.2
- net GND: now also C7.2, C9.2, R11.1, R14.1, R18.1, R22.1, R7.1, C34.2, C35.2, C42.1, C?.2, C?.2, C?.2, C?.2, C?.2, C?.2, C?.2, J3.4 (GND), J3.5 (Shield), J?.3 (Pin_3), J?.4 (GND), J?.5 (Shield), R?.1, R?.1, R?.2, U?.23 (GND), U?.35 (GND), U?.47 (GND), U?.8 (GND); no longer R10.1, R11.2, R14.2, R19.2, R20.1, SW1.2
- net N_RST: now also R20.1; no longer R18.1
- net OE1_FLAG: now also U12.9 (~DFLAG); no longer U11.9 (~DFLAG)
- net OE1_MISO: now also U12.6 (MISO); no longer U11.6 (MISO)
- net OE1_MOSI: now also U12.7 (MOSI); no longer U11.7 (MOSI)
- net OE1_SCK: now also U12.5 (SCK); no longer U11.5 (SCK)
- net OE1_SS: now also U12.4 (~SS); no longer U11.4 (~SS)
- net OE2_FLAG: now also U11.9 (~DFLAG); no longer U12.9 (~DFLAG)
- net OE2_MISO: now also U11.6 (MISO); no longer U12.6 (MISO)
- net OE2_MOSI: now also U11.7 (MOSI); no longer U12.7 (MOSI)
- net OE2_SCK: now also U11.5 (SCK); no longer U12.5 (SCK)
- net OE2_SS: now also U11.4 (~SS); no longer U12.4 (~SS)
- net SWD1_CLK: now also SW?.1 (A)
- net SWD1_IO: now also SW?.1 (A)
- net SWD2_CLK: now also SW?.3 (C)
- net SWD2_IO: now also SW?.3 (C)
- net at D3.2 (A), U4.8 (VBUS): now also C22.1, C23.1, U4.7 (REGIN), J3.1 (VBUS)
- net at U4.5 (DN): now also J3.2 (D-)
- net at U4.4 (DP): now also J3.3 (D+)
- net at D1.2 (A): now also SW2.2 (B)
- net at J2.1: now also SW2.1 (A)
- net at L1.1, U2.11 (PH): now also C14.1, U2.12 (PH)
- net at U2.7 (V_SNS): now also R10.1, R11.2; no longer R7.1
- net at U4.6 (VDD): now also C20.1
- net at D3.1 (K): now also R7.2; no longer R11.1
- net at J5.1 (Pin_1): now also R21.1; no longer R21.2
- net at J5.3 (Pin_3): now also R19.1; no longer R22.2
- net at U7.44 (BOOT0): now also R18.2; no longer R19.1
- net at D4.1 (K): now also R22.2; no longer R20.2
- net at L2.1, U6.13 (VDDA): now also C30.1, C35.1; no longer C33.1
- net at U6.30 (VCAP): now also C37.1; no longer C36.1
- net at U6.6 (PH1), Y2.2: now also C42.2
- net at U6.60 (BOOT0): now also R14.2; no longer R14.1
- new net: D?.1 (K), R?.2
- new net: C?.1, U?.5 (OSC_IN), Y?.1
- new net: C?.1, U?.6 (OSC_OUT), Y?.2
- new net: J?.2 (D-), U?.32 (PA11)
- new net: J?.3 (D+), R?.2, U?.33 (PA12)
- new net: R?.1, R?.2, U?.10 (PA0)
- new net: J?.1 (Pin_1), U?.30 (PA9)
- new net: J?.2 (Pin_2), U?.31 (PA10)
- new net: SW?.2 (B), U?.34 (SWD_IO)
- new net: SW?.2 (B), U?.37 (SWD_CLK)
- new net: R?.1, U?.44 (BOOT0)
- new net: C?.1, R?.1, U?.7 (NRST)

Commit message: PCB redrawing with correct net
Parts:
- removed C1, C11: 1u, Capacitors_SMD:C_0805_HandSoldering, symbol C
- removed C40, C43: 100n, Capacitors_SMD:C_0603_HandSoldering, symbol C
- removed C45: 0.1u, Capacitors_SMD:C_0805_HandSoldering, symbol C
- removed R17: 4K7, Resistors_SMD:R_0603_HandSoldering, symbol R
- added C13, C41, C42, C6: 100n, Capacitors_SMD:C_0603_HandSoldering, symbol C
- added C37: 1u, Capacitors_SMD:C_0805_HandSoldering, symbol C
- added C47: 0.1u, Capacitors_SMD:C_0603_HandSoldering, symbol C
- added R13: 4K7, Resistors_SMD:R_0603_HandSoldering, symbol R
- C12, C4: value 100n -> 1u; footprint Capacitors_SMD:C_0603_HandSoldering -> Capacitors_SMD:C_0805_HandSoldering
- J1: renamed from J?; footprint (none) -> Connectors_USB:USB_Micro-B_Molex_47346-0001
- J3: footprint (none) -> Connectors_USB:USB_Micro-B_Molex_47346-0001
- Q1: footprint TO_SOT_Packages_THT:TO-92_Inline_Narrow_Oval -> TO_SOT_Packages_THT:TO-92_Molded_Narrow
- R27: footprint Resistors_SMD:R_0603_HandSoldering -> Resistors_SMD:R_1210_HandSoldering
- R8: renamed from R7; value 2K2 -> 4K7
- RV1: value 10K -> POT; footprint Potentiometers:Potentiometer_Trimmer_ACP_CA14VSMD_Horizontal_Px13.0mm_Py10.0mm_MountLS -> Potentiometers:Potentiometer_Trimmer_ACP_CA14VSMD_Horizontal_Px13.0mm_Py10.0mm
- gave numbers to parts that had none: 19
- renumbered C2 to C1, C14 to C11, C13 to C14, C20 to C17, C21 to C19, C3 to C2, C22 to C20, C23 to C22, C31 to C28, C28 to C29, C7 to C3, C29 to C30, C34 to C31, C30 to C32, C32 to C33, C33 to C34, C36 to C35, C35 to C36, C37 to C40, C41 to C43, C42 to C44, C44 to C45, C47 to C48, C50 to C49, C9 to C5, C51 to C50, C48 to C51, C49 to C52, D3 to D2, J7 to J6, J6 to J7, R13 to R14, R14 to R17, R20 to R19, R3 to R2, R22 to R20, R19 to R21, R21 to R22, R26 to R25, R25 to R26, R10 to R6, R11 to R7, U12 to U11, U11 to U12, Y4 to Y3, Y3 to Y4
Connections:
- net +3.3VA: now also R3.1, C13.1; no longer R3.2
- net +3V3: now also C37.1, C41.1, R13.2
- net +5V: now also C42.1, C47.1
- net DISP_SCL: now also R13.1; no longer R15.1
- net DISP_SDA: now also R15.1
- net GND: now also SW1.2, C13.2, C37.2, C41.2, C42.2, C47.2, C6.2
- net VBUS: now reaches C4.1, U1.1 (VIN), U1.3 (INH)
- net VBUS: now also J1.1 (VBUS), C6.1
- net at SW1.1: now also C9.1, R3.2, U3.7 (NRST)
- net DN: now reaches J1.2 (D-), U3.32 (PA11)
- net DP: now reaches J1.3 (D+), R1.2, U3.33 (PA12)
Other:
- moved on the sheet: C1, C11, C14, C15, C16, C17, C18, C2, C20, C21, C22, C23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
